File: circuitos/circuito y placa/_autosave-circuito y placa.kicad_sch (KiCad schematic)
At the start: 9 parts, among them J1 aux, J2 MODULO, J4 PANTALLA, J5 B.ENCENDIDO, J6 B.PARADA, J7 LED Y BUFFER, J8 RELE

Commit message: negatico para imprecion
Parts:
- J1: footprint (none) -> Connector_PinHeader_1.00mm:PinHeader_1x02_P1.00mm_Vertical
Changed lines of the file:
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@@
 			)
 		)
-		(property "Footprint" ""
+		(property "Footprint" "Connector_PinHeader_1.00mm:PinHeader_1x02_P1.00mm_Vertical"
 			(at 156.21 55.88 0)
 			(effects
